File: hardware/badge_8.8_2024.kicad_sch (KiCad schematic)
At the start: 16 parts, among them J1 Conn_02x03_Odd_Even, SW1 SW_RST, SW2 On, U1 PY32F002AA15M6TU

Commit message: feat(Hw):Update_PCB
Parts:
- D1: value Green -> Orange; LCSC# C965815 -> C434437
- D4: value Orange -> Green; LCSC# C434437 -> C965815
Changed lines of the file:
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@@
 			)
 		)
-		(property "Value" "Orange"
+		(property "Value" "Green"
 			(at 182.753 87.884 0)
 			(effects
@@
 			)
 		)
-		(property "LCSC#" "C434437"
+		(property "LCSC#" "C965815"
 			(at 182.88 91.44 0)
 			(effects
@@
 			)
 		)
-		(property "Value" "Green"
+		(property "Value" "Orange"
 			(at 182.6895 58.166 0)
 			(effects
@@
 			)
 		)
-		(property "LCSC#" "C965815"
+		(property "LCSC#" "C434437"
 			(at 182.626 61.722 0)
 			(effects
