File: hardware/badge_8.8_2024.kicad_pcb (KiCad board)
At the start: 2 copper layers, 50 x 50 mm, 23 parts, among them J1 Conn_02x03_Odd_Even, SW1 SW_RST, SW2 On, U1 PY32F002AA15M6TU

Commit message: feat(Hw):Update_PCB
Parts:
- added kibuzzard-66ECA9F9: G***, kibuzzard-66ECA9F9, B.Cu at (68.8, 73.5)
- added kibuzzard-66ECAA39: G***, kibuzzard-66ECAA39, B.Cu at (68.8, 78.5)
- D1: value Green -> Orange
- D4: value Orange -> Green
Routing:
- net Net-(BT1--): track 20.5 -> 23.5 mm
- net /PA1: track 30.9 -> 32.0 mm

Commit message: feat(Hw):Add_label
Parts:
- added kibuzzard-66EDECB6: G***, kibuzzard-66EDECB6, B.Cu at (54.5, 43.5)
Changed lines of the file:
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@@
+		)
+	)
+	(footprint "kibuzzard-66EDECB6"
+		(layer "B.Cu")
+		(at 54.46 43.45 180)
+		(descr "Generated with KiBuzzard")
+		(tags "kb_params=eyJBbGlnbm1lbnRDaG9pY2UiOiAiQ2VudGVyIiwgIkNhcExlZnRDaG9pY2UiOiAiKCIsICJDYXBSaWdodENob2ljZSI6ICIpIiwgIkZvbnRDb21ib0JveCI6ICJVYnVudHVNb25vLUIiLCAiSGVpZ2h0Q3RybCI6IDEuMCwgIkxheWVyQ29tYm9Cb3giOiAiRi5TaWxrUyIsICJMaW5lU3BhY2luZ0N0cmwiOiAxLjUsICJNdWx0aUxpbmVUZXh0IjogInYxLjAiLCAiUGFkZGluZ0JvdHRvbUN0cmwiOiAxLjAsICJQYWRkaW5nTGVmdEN0cmwiOiAyLjUsICJQYWRkaW5nUmlnaHRDdHJsIjogMi41LCAiUGFkZGluZ1RvcEN0cmwiOiAxLjAsICJXaWR0aEN0cmwiOiAxLjB9")
+		(property "Reference" "kibuzzard-66EDECB6"
+			(at 0 3.676999 0)
+			(layer "B.SilkS")
+			(hide yes)
+			(effects
+				(font
+					(size 0.001 0.001)
+				)
+				(justify mirror)
+			)
+		)
+		(property "Value" "G***"
+			(at 0 -3.676999 0)
+			(layer "B.SilkS")
+			(hide yes)
+			(effects
+				(font
+					(size 0.001 0.001)
+				)
+				(justify mirror)
+			)
+		)
+		(property "Footprint" ""
+			(at 0 0 0)
+			(layer "B.Fab")
+			(hide yes)
+			(effects
+				(font
+					(size 1.27 1.27)
+					(thickness 0.15)
+				)
+				(justify mirror)
+			)
+		)
+		(property "Datasheet" ""
+			(at 0 0 0)
+			(layer "B.Fab")
+			(hide yes)
+			(effects
+				(font
+					(size 1.27 1.27)
+					(thickness 0.15)
+				)
+				(justify mirror)
+			)
+		)
+		(property "Description" ""
+			(at 0 0 0)
+			(layer "B.Fab")
+			(hide yes)
+			(effects
+				(font
+					(size 1.27 1.27)
+					(thickness 0.15)
+				)
+				(justify mirror)
+			)
+		)
+		(attr board_only exclude_from_pos_files exclude_from_bom)
+		(fp_poly
+			(pts
+				(xy 1.338235 0.001548) (xy 1.333677 0.102253) (xy 1.320003 0.185587) (xy 1.297214 0.251548) (xy 1.246711 0.315983)
+				(xy 1.177245 0.337461) (xy 1.108746 0.315983) (xy 1.05805 0.251548) (xy 1.03483 0.185587) (xy 1.020898 0.102253)
+				(xy 1.016254 0.001548) (xy 1.020898 -0.100017) (xy 1.03483 -0.183867) (xy 1.05805 -0.25) (xy 1.108746 -0.314435)
+				(xy 1.177245 -0.335913) (xy 1.178793 -0.335435) (xy 1.178793 -0.085139) (xy 1.115325 -0.054954)
+				(xy 1.092105 0.017028) (xy 1.115325 0.089783) (xy 1.178793 0.120743) (xy 1.239938 0.089783) (xy 1.263932 0.017028)
+				(xy 1.239938 -0.054954) (xy 1.178793 -0.085139) (xy 1.178793 -0.335435) (xy 1.246711 -0.314435)
+				(xy 1.297214 -0.25) (xy 1.320003 -0.183867) (xy 1.333677 -0.100017) (xy 1.338235 0.001548)
+			)
+			(stroke
+				(width 0)
+				(type solid)
+			)
+			(fill solid)
+			(layer "B.SilkS")
+		)
+		(fp_poly
+			(pts
+				(xy -1.510062 0.628999) (xy -1.832559 0.628999) (xy -1.955271 0.616913) (xy -2.073267 0.581119)
+				(xy -2.182012 0.522994) (xy -2.277329 0.444769) (xy -2.355553 0.349453) (xy -2.413679 0.240707)
+				(xy -2.449472 0.122712) (xy -2.461558 0) (xy -2.449472 -0.122712) (xy -2.413679 -0.240707) (xy -2.355553 -0.349453)
+				(xy -2.277329 -0.444769) (xy -2.182012 -0.522994) (xy -2.073267 -0.581119) (xy -1.955271 -0.616913)
+				(xy -1.832559 -0.628999) (xy -1.510062 -0.628999) (xy -1.231424 -0.628999) (xy -1.231424 -0.479876)
+				(xy -1.278122 -0.382783) (xy -1.325335 -0.275198) (xy -1.373065 -0.157121) (xy -1.40862 -0.062452)
+				(xy -1.443305 0.036571) (xy -1.477119 0.139948) (xy -1.510062 0.247678) (xy -1.310372 0.247678)
+				(xy -1.295085 0.18692) (xy -1.27709 0.122291) (xy -1.257159 0.055534) (xy -1.236068 -0.01161) (xy -1.214203 -0.07798)
+				(xy -1.19195 -0.142415) (xy -1.149381 -0.258514) (xy -1.104489 -0.142415) (xy -1.079915 -0.07798)
+				(xy -1.055728 -0.01161) (xy -1.032121 0.055534) (xy -1.009288 0.122291) (xy -0.988971 0.18692) (xy -0.97291 0.247678)
+				(xy -0.779412 0.247678) (xy -0.81279 0.139948) (xy -0.84791 0.036571) (xy -0.884772 -0.062452) (xy -0.923375 -0.157121)
+				(xy -0.974974 -0.275198) (xy -1.02451 -0.382783) (xy -1.071981 -0.479876) (xy -1.231424 -0.479876)
+				(xy -1.231424 -0.628999) (xy -0.047214 -0.628999) (xy -0.047214 -0.479876) (xy -0.629257 -0.479876)
+				(xy -0.629257 -0.321981) (xy -0.428019 -0.321981) (xy -0.428019 0.213622) (xy -0.52709 0.158669)
+				(xy -0.621517 0.120743) (xy -0.683437 0.278638) (xy -0.602941 0.314241) (xy -0.516254 0.362229)
+				(xy -0.434211 0.417957) (xy -0.367647 0.478328) (xy -0.237616 0.478328) (xy -0.237616 -0.321981)
+				(xy -0.047214 -0.321981) (xy -0.047214 -0.479876) (xy -0.047214 -0.628999) (xy 0.404799 -0.628999)
+				(xy 0.404799 -0.496904) (xy 0.352167 -0.487616) (xy 0.30805 -0.460526) (xy 0.27709 -0.417183) (xy 0.26548 -0.357585)
+				(xy 0.27709 -0.299536) (xy 0.30805 -0.256966) (xy 0.352167 -0.23065) (xy 0.404799 -0.221362) (xy 0.500774 -0.256966)
+				(xy 0.54257 -0.357585) (xy 0.500774 -0.4613) (xy 0.404799 -0.496904) (xy 0.404799 -0.628999) (xy 1.177245 -0.628999)
+				(xy 1.177245 -0.5) (xy 1.077485 -0.48624) (xy 0.994926 -0.44496) (xy 0.929567 -0.376161) (xy 0.892318 -0.306115)
+				(xy 0.865712 -0.219814) (xy 0.849748 -0.11726) (xy 0.844427 0.001548) (xy 0.849845 0.119002) (xy 0.866099 0.220588)
+				(xy 0.893189 0.306308) (xy 0.931115 0.376161) (xy 0.99699 0.44496) (xy 1.079033 0.48624) (xy 1.177245 0.5)
+				(xy 1.277004 0.486326) (xy 1.359563 0.445304) (xy 1.424923 0.376935) (xy 1.462171 0.307324) (xy 1.488777 0.221556)
+				(xy 1.504741 0.11963) (xy 1.510062 0.001548) (xy 1.504741 -0.11726) (xy 1.488777 -0.219814) (xy 1.462171 -0.306115)
+				(xy 1.424923 -0.376161) (xy 1.359563 -0.44496) (xy 1.277004 -0.48624) (xy 1.177245 -0.5) (xy 1.177245 -0.628999)
+				(xy 1.510062 -0.628999) (xy 1.832559 -0.628999) (xy 1.955271 -0.616913) (xy 2.073267 -0.581119)
+				(xy 2.182012 -0.522994) (xy 2.277329 -0.444769) (xy 2.355553 -0.349453) (xy 2.413679 -0.240707)
+				(xy 2.449472 -0.122712) (xy 2.461558 0) (xy 2.449472 0.122712) (xy 2.413679 0.240707) (xy 2.355553 0.349453)
+				(xy 2.277329 0.444769) (xy 2.182012 0.522994) (xy 2.073267 0.581119) (xy 1.955271 0.616913) (xy 1.832559 0.628999)
+				(xy 1.510062 0.628999) (xy -1.510062 0.628999)
+			)
+			(stroke
+				(width 0)
+				(type solid)
+			)
+			(fill solid)
+			(layer "B.SilkS")
 		)
 	)
@@
 				(font
 					(size 0.001 0.001)
+					(thickness 0.15)
 				)
 				(justify mirror)
@@
 				(font
 					(size 0.001 0.001)
+					(thickness 0.15)
 				)
 				(justify mirror)
@@
 				(font
 					(size 0.001 0.001)
+					(thickness 0.15)
 				)
 				(justify mirror)
@@
 				(font
 					(size 0.001 0.001)
-				)
-				(justify mirror)
+					(thickness 0.15)
+				)
+				(justify mirror)

Commit message: feat(Hw):Add_labels
Other:
- board text added: "https://youtu.be/ dQw4w9WgXcQ?si=N 39gOwTvt6YGSlYW"
Changed lines of the file:
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@@
 				(font
 					(size 0.001 0.001)
+					(thickness 0.15)
 				)
 				(justify mirror)
@@
 				(font
 					(size 0.001 0.001)
+					(thickness 0.15)
 				)
 				(justify mirror)
@@
 		(layer "Edge.Cuts")
 	)
+	(gr_text "https://youtu.be/\ndQw4w9WgXcQ?si=N\n39gOwTvt6YGSlYW"
+		(at 49.67 65.35 0)
+		(layer "B.SilkS")
+		(effects
+			(font
+				(size 1 1)
+				(thickness 0.15)
+			)
+			(justify mirror)
+		)
+	)
 	(segment

Commit message: feat(Hw):Update_Labeles
Parts:
- added G***: LOGO, Library:qr, B.Cu at (49.5, 65.0)
Other:
- board text removed: "https://youtu.be/ dQw4w9WgXcQ?si=N 39gOwTvt6YGSlYW"

Commit message: feat(Hw):Update_Lables
Parts:
- moved G*** 1.48 mm to (49.1, 66.4)
